Commit message: feat: implement universal PID node, robust world baking, and cascaded control lab

File: src/pid_controller_pkg/urdf/single_pendulum.urdf (robot description, URDF)
Before this commit: robot sliding_double_pendulum, 7 links, 6 joints
Links:
- removed link arm_2_link
- removed link sensor_frame
- removed link target_marker
Joints:
- removed joint pendulum_2_joint
- removed joint slider_to_sensor
- removed joint world_to_target
- joint pendulum_joint: origin xyz=0 0 0 rpy=3.14 0 0 -> xyz=0 0 0 rpy=3.15 0 0
